File: 2001captchpad.sch (KiCad schematic (older format))
At the start: 21 parts, among them J1 TIP, J2 GND, J3 RING, J4 DIT, J5 DAH, J6 +, J7 -, Q1 IRFML8244TRPBF, Q2 IRFML8244TRPBF, U1 AT42QT1011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

Commit message: Updated 20191229
Parts:
- Q1, Q2: symbol 2001captchpad-rescue:IRFML8244TRPBF-IRFML8244TRPBF -> IRFML8244TRPBF:IRFML8244TRPBF
Changed lines of the file:
@@
 $EndDescr
 $Comp
-L 2001captchpad-rescue:IRFML8244TRPBF-IRFML8244TRPBF Q1
+L IRFML8244TRPBF:IRFML8244TRPBF Q1
 U 1 1 5DEB371A
 P 4300 2800
@@
 $EndComp
 $Comp
-L 2001captchpad-rescue:IRFML8244TRPBF-IRFML8244TRPBF Q2
+L IRFML8244TRPBF:IRFML8244TRPBF Q2
 U 1 1 5DEB37DE
 P 4250 4350

Commit message: Mirrored schematic
Parts:
- Q1, Q2: symbol IRFML8244TRPBF:IRFML8244TRPBF -> 2001captchpad-rescue:IRFML8244TRPBF-IRFML8244TRPBF
Other:
- moved on the sheet: C1, C2, C3, C4, H1, H2, H3, H4, J1, J2, J3, J4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
